Commit message: mr_rehri_all plugins added

File: mr_rehri/urdf/1_simple_rehri.urdf (robot description, URDF)
Before this commit: robot rehri, 4 links, 3 joints
Links:
- added link base_footprint
Joints:
- added joint base_joint: type fixed, parent base_footprint, child base, origin xyz=0 0 0.135 rpy=0 0 0

File: mr_rehri/urdf/2_gazebo_diff_drive.urdf (robot description, URDF)
Before this commit: robot rehri, 4 links, 3 joints
Links:
- added link base_footprint
Joints:
- added joint base_joint: type fixed, parent base_footprint, child base, origin xyz=0 0 0.135 rpy=0 0 0
